Commit message: project 4

File: src/my_robot/urdf/my_robot.xacro (robot description, xacro)
@@ -133,5 +133,5 @@
         <dynamic damping="1.0" friction="1.0"/>
       </joint>
-      <link name="camera">
+      <link name="camera_link_optical">
         <inertial>
           <mass value="0.1"/>
@@ -159,9 +159,8 @@
         </visual>
       </link>
-      <joint name="camera_joint" type="fixed">
-        <origin xyz="0.225 0 0" rpy="0 0 0" />
+      <joint name="camera_optical_joint" type="fixed">
+        <origin xyz="0.17 0 0.025" rpy="-1.5707 0 -1.5707"/>
         <parent link="chassis"/>
-        <child link="camera" />
-        <axis xyz="0 1 0" rpy="0 0 0"/>
+        <child link="camera_link_optical"/>
       </joint>
       <link name="hokuyo">

File: src/turtlebot/turtlebot_description/robots/create_circles_asus_xtion_pro.urdf.xacro (robot description, xacro)
@@ -9,7 +9,7 @@
   <xacro:include filename="$(find create_description)/urdf/create.urdf.xacro"/>
   <xacro:include filename="$(find turtlebot_description)/urdf/stacks/circles.urdf.xacro"/>
-  <xacro:include filename="$(find turtlebot_description)/urdf/sensors/xtion_pro.urdf.xacro"/>
-  <xacro:create/>
-  <xacro:stack_circles    parent="base_link"/>
-  <xacro:sensor_xtion_pro parent="base_link"/>
+  <xacro:include filename="$(find turtlebot_description)/urdf/sensors/asus_xtion_pro.urdf.xacro"/>
+  <create/>
+  <stack_circles parent="base_link"/>
+  <sensor_asus_xtion_pro  parent="base_link"/>
 </robot>

File: src/turtlebot/turtlebot_description/robots/create_circles_kinect.urdf.xacro (robot description, xacro)
@@ -10,6 +10,6 @@
   <xacro:include filename="$(find turtlebot_description)/urdf/stacks/circles.urdf.xacro"/>
   <xacro:include filename="$(find turtlebot_description)/urdf/sensors/kinect.urdf.xacro"/>
-  <xacro:create/>
-  <xacro:stack_circles parent="base_link"/>
-  <xacro:sensor_kinect parent="base_link"/>
+  <create/>
+  <stack_circles parent="base_link"/>
+  <sensor_kinect  parent="base_link"/>
 </robot>

File: src/turtlebot/turtlebot_description/robots/kobuki_hexagons_astra.urdf.xacro (robot description, xacro)
@@ -10,6 +10,6 @@
   <xacro:include filename="$(find turtlebot_description)/urdf/stacks/hexagons.urdf.xacro"/>
   <xacro:include filename="$(find turtlebot_description)/urdf/sensors/astra.urdf.xacro"/>
-  <xacro:kobuki/>
-  <xacro:stack_hexagons parent="base_link"/>
-  <xacro:sensor_astra   parent="base_link"/>
+  <kobuki/>
+  <stack_hexagons parent="base_link"/>
+  <sensor_astra parent="base_link"/>
 </robot>

File: src/turtlebot/turtlebot_description/robots/kobuki_hexagons_asus_xtion_pro.urdf.xacro (robot description, xacro)
@@ -9,7 +9,7 @@
   <xacro:include filename="$(find kobuki_description)/urdf/kobuki.urdf.xacro" />
   <xacro:include filename="$(find turtlebot_description)/urdf/stacks/hexagons.urdf.xacro"/>
-  <xacro:include filename="$(find turtlebot_description)/urdf/sensors/xtion_pro.urdf.xacro"/>
-  <xacro:kobuki/>
-  <xacro:stack_hexagons   parent="base_link"/>
-  <xacro:sensor_xtion_pro parent="base_link" xtion_pro_cam_py="0.0205"/>
+  <xacro:include filename="$(find turtlebot_description)/urdf/sensors/asus_xtion_pro.urdf.xacro"/>
+  <kobuki/>
+  <stack_hexagons                 parent="base_link"/>
+  <sensor_asus_xtion_pro          parent="base_link"/>
 </robot>

File: src/turtlebot/turtlebot_description/robots/kobuki_hexagons_asus_xtion_pro_offset.urdf.xacro (robot description, xacro)
@@ -9,7 +9,7 @@
   <xacro:include filename="$(find kobuki_description)/urdf/kobuki.urdf.xacro" />
   <xacro:include filename="$(find turtlebot_description)/urdf/stacks/hexagons.urdf.xacro"/>
-  <xacro:include filename="$(find turtlebot_description)/urdf/sensors/xtion_pro.urdf.xacro"/>
-  <xacro:kobuki/>
-  <xacro:stack_hexagons   parent="base_link"/>
-  <xacro:sensor_xtion_pro parent="base_link" xtion_pro_cam_py="-0.0125"/>
+  <xacro:include filename="$(find turtlebot_description)/urdf/sensors/asus_xtion_pro_offset.urdf.xacro"/>
+  <kobuki/>
+  <stack_hexagons                 parent="base_link"/>
+  <sensor_asus_xtion_pro_offset   parent="base_link"/>
 </robot>

File: src/turtlebot/turtlebot_description/robots/kobuki_hexagons_kinect.urdf.xacro (robot description, xacro)
@@ -10,6 +10,6 @@
   <xacro:include filename="$(find turtlebot_description)/urdf/stacks/hexagons.urdf.xacro"/>
   <xacro:include filename="$(find turtlebot_description)/urdf/sensors/kinect.urdf.xacro"/>
-  <xacro:kobuki/>
-  <xacro:stack_hexagons parent="base_link"/>
-  <xacro:sensor_kinect parent="base_link"/>
+  <kobuki/>
+  <stack_hexagons parent="base_link"/>
+  <sensor_kinect  parent="base_link"/>
 </robot>

File: src/turtlebot/turtlebot_description/robots/kobuki_hexagons_r200.urdf.xacro (robot description, xacro)
@@ -10,6 +10,6 @@
   <xacro:include filename="$(find turtlebot_description)/urdf/stacks/hexagons.urdf.xacro"/>
   <xacro:include filename="$(find turtlebot_description)/urdf/sensors/r200.urdf.xacro"/>
-  <xacro:kobuki/>
-  <xacro:stack_hexagons parent="base_link"/>
-  <xacro:sensor_r200    parent="base_link"/>
+  <kobuki/>
+  <stack_hexagons parent="base_link"/>
+  <sensor_r200  parent="base_link"/>
 </robot>

File: src/turtlebot/turtlebot_description/urdf/sensors/astra.urdf.xacro (robot description, xacro)
@@ -63,5 +63,5 @@
     <link name="camera_depth_optical_frame"/>
     <!-- RGBD sensor for simulation, same as Kinect -->
-    <xacro:turtlebot_sim_3dsensor/>
+    <turtlebot_sim_3dsensor/>
   </xacro:macro>
 </robot>

File: src/turtlebot/turtlebot_description/urdf/sensors/kinect.urdf.xacro (robot description, xacro)
@@ -60,5 +60,5 @@
 	<link name="camera_depth_optical_frame"/>
 	<!-- Kinect sensor for simulation -->
-	<xacro:turtlebot_sim_3dsensor/>
+	<turtlebot_sim_3dsensor/>
   </xacro:macro>
 </robot>

File: src/turtlebot/turtlebot_description/urdf/sensors/r200.urdf.xacro (robot description, xacro)
@@ -129,5 +129,5 @@
     <link name="camera_depth_optical_frame"/>
   	<!-- Simulation sensor -->
-    <xacro:turtlebot_sim_3dsensor/>
+    <turtlebot_sim_3dsensor/>
   </xacro:macro>
 </robot>

File: src/turtlebot/turtlebot_description/urdf/stacks/circles.urdf.xacro (robot description, xacro)
@@ -142,8 +142,8 @@
   </xacro:macro>
   <xacro:macro name="stack_circles" params="parent">
-    <xacro:turtlebot_spacer parent="${parent}" number="0" x_loc="-0.00254" y_loc="0.1114679" z_loc="0.062992"/>
-    <xacro:turtlebot_spacer parent="${parent}" number="1" x_loc="-0.00254" y_loc="-0.1114679" z_loc="0.062992"/>
-    <xacro:turtlebot_spacer parent="${parent}" number="2" x_loc="-0.07239" y_loc="-0.1114679" z_loc="0.062992"/>
-    <xacro:turtlebot_spacer parent="${parent}" number="3" x_loc="-0.07239" y_loc="0.1114679" z_loc="0.062992"/>
+    <turtlebot_spacer parent="${parent}" number="0" x_loc="-0.00254" y_loc="0.1114679" z_loc="0.062992"/>
+    <turtlebot_spacer parent="${parent}" number="1" x_loc="-0.00254" y_loc="-0.1114679" z_loc="0.062992"/>
+    <turtlebot_spacer parent="${parent}" number="2" x_loc="-0.07239" y_loc="-0.1114679" z_loc="0.062992"/>
+    <turtlebot_spacer parent="${parent}" number="3" x_loc="-0.07239" y_loc="0.1114679" z_loc="0.062992"/>
     <joint name="plate_0_joint" type="fixed">
       <origin xyz="-0.04334 0  0.06775704" rpy="0 0 0" />
@@ -172,8 +172,8 @@
       </collision>
     </link>
-    <xacro:turtlebot_standoff_2in parent="${parent}" number="0" x_loc="0.0676402" y_loc="0.1314196" z_loc="0.0709803"/>
-    <xacro:turtlebot_standoff_2in parent="${parent}" number="1" x_loc="0.0676402" y_loc="-0.1314196" z_loc="0.0709803"/>
-    <xacro:turtlebot_standoff_2in parent="${parent}" number="2" x_loc="-0.052832" y_loc="-0.1314196" z_loc="0.0709803"/>
-    <xacro:turtlebot_standoff_2in parent="${parent}" number="3" x_loc="-0.052832" y_loc="0.1314196" z_loc="0.0709803"/>
+    <turtlebot_standoff_2in parent="${parent}" number="0" x_loc="0.0676402" y_loc="0.1314196" z_loc="0.0709803"/>
+    <turtlebot_standoff_2in parent="${parent}" number="1" x_loc="0.0676402" y_loc="-0.1314196" z_loc="0.0709803"/>
+    <turtlebot_standoff_2in parent="${parent}" number="2" x_loc="-0.052832" y_loc="-0.1314196" z_loc="0.0709803"/>
+    <turtlebot_standoff_2in parent="${parent}" number="3" x_loc="-0.052832" y_loc="0.1314196" z_loc="0.0709803"/>
     <joint name="plate_1_joint" type="fixed">
       <origin xyz="0.04068 0 0.05715" rpy="0 0 0" />
@@ -202,8 +202,8 @@
       </collision>
     </link>
-    <xacro:turtlebot_standoff_2in parent="standoff_2in_0_link" number="4" x_loc="0" y_loc="0" z_loc="0.05715"/>
-    <xacro:turtlebot_standoff_2in parent="standoff_2in_1_link" number="5" x_loc="0" y_loc="0" z_loc="0.05715"/>
-    <xacro:turtlebot_standoff_2in parent="standoff_2in_2_link" number="6" x_loc="0" y_loc="0" z_loc="0.05715"/>
-    <xacro:turtlebot_standoff_2in parent="standoff_2in_3_link" number="7" x_loc="0" y_loc="0" z_loc="0.05715"/>
+    <turtlebot_standoff_2in parent="standoff_2in_0_link" number="4" x_loc="0" y_loc="0" z_loc="0.05715"/>
+    <turtlebot_standoff_2in parent="standoff_2in_1_link" number="5" x_loc="0" y_loc="0" z_loc="0.05715"/>
+    <turtlebot_standoff_2in parent="standoff_2in_2_link" number="6" x_loc="0" y_loc="0" z_loc="0.05715"/>
+    <turtlebot_standoff_2in parent="standoff_2in_3_link" number="7" x_loc="0" y_loc="0" z_loc="0.05715"/>
     <joint name="plate_2_joint" type="fixed">
       <origin xyz="0 0 0.0572008" rpy="0 0 0" />
@@ -232,10 +232,10 @@
       </collision>
     </link>
-    <xacro:turtlebot_standoff_kinect parent="plate_2_link" number="0" x_loc="-0.1024382" y_loc="0.098" z_loc="0.0032004"/>
-    <xacro:turtlebot_standoff_kinect parent="plate_2_link" number="1" x_loc="-0.1024382" y_loc="-0.098" z_loc="0.0032004"/>
-    <xacro:turtlebot_standoff_8in parent="standoff_2in_4_link" number="0" x_loc="0" y_loc="0" z_loc="0.05715"/>
-    <xacro:turtlebot_standoff_8in parent="standoff_2in_5_link" number="1" x_loc="0" y_loc="0" z_loc="0.05715"/>
-    <xacro:turtlebot_standoff_8in parent="standoff_2in_6_link" number="2" x_loc="0" y_loc="0" z_loc="0.05715"/>
-    <xacro:turtlebot_standoff_8in parent="standoff_2in_7_link" number="3" x_loc="0" y_loc="0" z_loc="0.05715"/>
+    <turtlebot_standoff_kinect parent="plate_2_link" number="0" x_loc="-0.1024382" y_loc="0.098" z_loc="0.0032004"/>
+    <turtlebot_standoff_kinect parent="plate_2_link" number="1" x_loc="-0.1024382" y_loc="-0.098" z_loc="0.0032004"/>
+    <turtlebot_standoff_8in parent="standoff_2in_4_link" number="0" x_loc="0" y_loc="0" z_loc="0.05715"/>
+    <turtlebot_standoff_8in parent="standoff_2in_5_link" number="1" x_loc="0" y_loc="0" z_loc="0.05715"/>
+    <turtlebot_standoff_8in parent="standoff_2in_6_link" number="2" x_loc="0" y_loc="0" z_loc="0.05715"/>
+    <turtlebot_standoff_8in parent="standoff_2in_7_link" number="3" x_loc="0" y_loc="0" z_loc="0.05715"/>
     <joint name="plate_3_joint" type="fixed">
       <origin xyz="-0.01316 0 0.2063496" rpy="0 0 0" />

File: src/turtlebot/turtlebot_description/urdf/stacks/hexagons.urdf.xacro (robot description, xacro)
@@ -9,7 +9,7 @@
   <!-- Xacro macros -->
   <!-- Pole macros -->
-  <xacro:macro name="stack_bottom_pole" params="parent number x_loc y_loc z_loc roll=0.0 pitch=0.0 yaw=0.0">
+  <xacro:macro name="stack_bottom_pole" params="parent number x_loc y_loc z_loc">
     <joint name="pole_bottom_${number}_joint" type="fixed">
-      <origin xyz="${x_loc} ${y_loc} ${z_loc}" rpy="${roll} ${pitch} ${yaw}"/>
+      <origin xyz="${x_loc} ${y_loc} ${z_loc}" rpy="0 0 0"/>
       <parent link="${parent}"/>
       <child link="pole_bottom_${number}_link"/>
@@ -37,7 +37,7 @@
     </link>
   </xacro:macro>
-  <xacro:macro name="stack_middle_pole" params="parent number x_loc y_loc z_loc roll=0.0 pitch=0.0 yaw=0.0">
+  <xacro:macro name="stack_middle_pole" params="parent number x_loc y_loc z_loc">
     <joint name="pole_middle_${number}_joint" type="fixed">
-      <origin xyz="${x_loc} ${y_loc} ${z_loc}" rpy="${roll} ${pitch} ${yaw}" />
+      <origin xyz="${x_loc} ${y_loc} ${z_loc}" rpy="0 0 0" />
       <parent link="${parent}"/>
       <child link="pole_middle_${number}_link"/>
@@ -65,7 +65,7 @@
     </link>
   </xacro:macro>
-  <xacro:macro name="stack_top_pole" params="parent number x_loc y_loc z_loc roll=0.0 pitch=0.0 yaw=0.0">
+  <xacro:macro name="stack_top_pole" params="parent number x_loc y_loc z_loc">
     <joint name="pole_top_${number}_joint" type="fixed">
-      <origin xyz="${x_loc} ${y_loc} ${z_loc}" rpy="${roll} ${pitch} ${yaw}"/>
+      <origin xyz="${x_loc} ${y_loc} ${z_loc}" rpy="0 0 0"/>
       <parent link="${parent}"/>
       <child link="pole_top_${number}_link"/>
@@ -93,7 +93,7 @@
     </link>
   </xacro:macro>
-  <xacro:macro name="stack_3d_sensor_pole" params="parent number x_loc y_loc z_loc roll=0.0 pitch=0.0 yaw=0.0">
+  <xacro:macro name="stack_3d_sensor_pole" params="parent number x_loc y_loc z_loc">
     <joint name="pole_kinect_${number}_joint" type="fixed">
-      <origin xyz="${x_loc} ${y_loc} ${z_loc}" rpy="${roll} ${pitch} ${yaw}"/>
+      <origin xyz="${x_loc} ${y_loc} ${z_loc}" rpy="0 0 0"/>
       <parent link="${parent}"/>
       <child link="pole_kinect_${number}_link"/>
@@ -101,7 +101,7 @@
     <link name="pole_kinect_${number}_link">
       <visual>
-        <origin xyz="0 0 0" rpy="0 0 0"/>
-        <geometry>
-          <mesh filename="package://turtlebot_description/meshes/stacks/hexagons/pole_kinect.dae" />
+        <origin xyz="0 0 -0.01" rpy="0 0 0"/>
+        <geometry>
+          <mesh filename="package://turtlebot_description/meshes/sensors/sensor_pole.dae" />
         </geometry>
       </visual>
@@ -127,10 +127,10 @@
   -->
   <xacro:macro name="stack_hexagons" params="parent">
-    <xacro:stack_bottom_pole parent="${parent}" number="0" x_loc= "0.120" y_loc= "0.082" z_loc="0.1028"/>
-    <xacro:stack_bottom_pole parent="${parent}" number="1" x_loc= "0.055" y_loc= "0.120" z_loc="0.1028"/>
-    <xacro:stack_bottom_pole parent="${parent}" number="2" x_loc="-0.055" y_loc= "0.120" z_loc="0.1028"/>
-    <xacro:stack_bottom_pole parent="${parent}" number="3" x_loc= "0.120" y_loc="-0.082" z_loc="0.1028"/>
-    <xacro:stack_bottom_pole parent="${parent}" number="4" x_loc= "0.055" y_loc="-0.120" z_loc="0.1028"/>
-    <xacro:stack_bottom_pole parent="${parent}" number="5" x_loc="-0.055" y_loc="-0.120" z_loc="0.1028"/>
+    <stack_bottom_pole parent="${parent}" number="0" x_loc= "0.120" y_loc= "0.082" z_loc="0.1028"/>
+    <stack_bottom_pole parent="${parent}" number="1" x_loc= "0.055" y_loc= "0.120" z_loc="0.1028"/>
+    <stack_bottom_pole parent="${parent}" number="2" x_loc="-0.055" y_loc= "0.120" z_loc="0.1028"/>
+    <stack_bottom_pole parent="${parent}" number="3" x_loc= "0.120" y_loc="-0.082" z_loc="0.1028"/>
+    <stack_bottom_pole parent="${parent}" number="4" x_loc= "0.055" y_loc="-0.120" z_loc="0.1028"/>
+    <stack_bottom_pole parent="${parent}" number="5" x_loc="-0.055" y_loc="-0.120" z_loc="0.1028"/>
     <joint name="plate_bottom_joint" type="fixed">
       <origin xyz="0.02364 0.0 0.1306" rpy="0 0 0"/>
@@ -159,8 +159,8 @@
       </inertial>
     </link>
-    <xacro:stack_middle_pole parent="${parent}" number="0" x_loc= "0.0381" y_loc= "0.1505" z_loc="0.1640"/>
-    <xacro:stack_middle_pole parent="${parent}" number="1" x_loc= "0.0381" y_loc="-0.1505" z_loc="0.1640"/>
-    <xacro:stack_middle_pole parent="${parent}" number="2" x_loc="-0.0381" y_loc= "0.1505" z_loc="0.1640"/>
-    <xacro:stack_middle_pole parent="${parent}" number="3" x_loc="-0.0381" y_loc="-0.1505" z_loc="0.1640"/>
+    <stack_middle_pole parent="${parent}" number="0" x_loc= "0.0381" y_loc= "0.1505" z_loc="0.1640"/>
+    <stack_middle_pole parent="${parent}" number="1" x_loc= "0.0381" y_loc="-0.1505" z_loc="0.1640"/>
+    <stack_middle_pole parent="${parent}" number="2" x_loc="-0.0381" y_loc= "0.1505" z_loc="0.1640"/>
+    <stack_middle_pole parent="${parent}" number="3" x_loc="-0.0381" y_loc="-0.1505" z_loc="0.1640"/>
     <joint name="plate_middle_joint" type="fixed">
       <origin xyz="-0.01364 0.0 0.1874" rpy="0 0 0"/>
@@ -178,6 +178,5 @@
         <origin xyz="0.01364 0.0 0.0" rpy="0 0 0"/>
         <geometry>
-          <mesh filename="package://turtlebot_description/meshes/stacks/hexagons/plate_simple.stl"
-                scale="${M_SCALE} ${M_SCALE} ${M_SCALE}"/>
+          <cylinder length="0.006" radius="0.170"/>
         </geometry>
       </collision>
@@ -190,10 +189,10 @@
       </inertial>
     </link>
-    <xacro:stack_top_pole parent="${parent}" number="0" x_loc= "0.0381" y_loc= "0.1505" z_loc="0.2920"/>
-    <xacro:stack_top_pole parent="${parent}" number="1" x_loc= "0.0381" y_loc="-0.1505" z_loc="0.2920"/>
-    <xacro:stack_top_pole parent="${parent}" number="2" x_loc="-0.0381" y_loc= "0.1505" z_loc="0.2920"/>
-    <xacro:stack_top_pole parent="${parent}" number="3" x_loc="-0.0381" y_loc="-0.1505" z_loc="0.2920"/>
-    <xacro:stack_3d_sensor_pole parent="${parent}" number="0" x_loc="-0.1024" y_loc= "0.098" z_loc="0.2372"/>
-    <xacro:stack_3d_sensor_pole parent="${parent}" number="1" x_loc="-0.1024" y_loc="-0.098" z_loc="0.2372"/>
+    <stack_top_pole parent="${parent}" number="0" x_loc= "0.0381" y_loc= "0.1505" z_loc="0.2920"/>
+    <stack_top_pole parent="${parent}" number="1" x_loc= "0.0381" y_loc="-0.1505" z_loc="0.2920"/>
+    <stack_top_pole parent="${parent}" number="2" x_loc="-0.0381" y_loc= "0.1505" z_loc="0.2920"/>
+    <stack_top_pole parent="${parent}" number="3" x_loc="-0.0381" y_loc="-0.1505" z_loc="0.2920"/>
+    <stack_3d_sensor_pole parent="${parent}" number="0" x_loc="-0.1024" y_loc= "0.098" z_loc="0.2372"/>
+    <stack_3d_sensor_pole parent="${parent}" number="1" x_loc="-0.1024" y_loc="-0.098" z_loc="0.2372"/>
     <joint name="plate_top_joint" type="fixed">
       <origin xyz="-0.01364 0.0  0.3966" rpy="0 0 0"/>
@@ -211,6 +210,5 @@
         <origin xyz="0.01364 0 0" rpy="0 0 0"/>
         <geometry>
-          <mesh filename="package://turtlebot_description/meshes/stacks/hexagons/plate_simple.stl"
-                scale="${M_SCALE} ${M_SCALE} ${M_SCALE}"/>
+          <cylinder length="0.006" radius="0.170"/>
         </geometry>
       </collision>

Commit message: Course 4: Map my world

File: src/my_robot/urdf/my_robot.xacro (robot description, xacro)
@@ -160,5 +160,5 @@
       </link>
       <joint name="camera_optical_joint" type="fixed">
-        <origin xyz="0.17 0 0.025" rpy="-1.5707 0 -1.5707"/>
+        <origin xyz="0.17 0 0.025" rpy="0 0 0"/>
         <parent link="chassis"/>
         <child link="camera_link_optical"/>

Commit message: Fix camera orientation

File: src/my_robot/urdf/my_robot.xacro (robot description, xacro)
@@ -133,5 +133,5 @@
         <dynamic damping="1.0" friction="1.0"/>
       </joint>
-      <link name="camera_link_optical">
+      <link name="camera">
         <inertial>
           <mass value="0.1"/>
@@ -159,9 +159,17 @@
         </visual>
       </link>
+      <joint name="camera_joint" type="fixed">
+        <origin xyz="0.225 0 0" rpy="0 0 0" />
+        <parent link="chassis"/>
+        <child link="camera" />
+        <axis xyz="0 1 0" rpy="0 0 0"/>
+      </joint>
       <joint name="camera_optical_joint" type="fixed">
-        <origin xyz="0.17 0 0.025" rpy="0 0 0"/>
-        <parent link="chassis"/>
-        <child link="camera_link_optical"/>
-      </joint>
+        <origin xyz="0 0 0" rpy="-1.5707 0 -1.5707" />
+        <parent link="camera"/>
+        <child link="camera_link_optical" />
+      </joint>
+      <link name="camera_link_optical">
+      </link>
       <link name="hokuyo">
       <inertial>
